File: Hardware/displayDriver.kicad_sch (KiCad schematic)
At the start: 1 part, among them U9 5082-7300

Commit message: chore: Finilize circuit parity
Add colon LEDs
Reannotate reference designations
Update footprints

Signed-off-by: Joel Cranmer <42.joel.cranmer@gmail.com>
Parts:
- U9: footprint (none) -> JKC_Library:Display_HP_5082-7300
Changed lines of the file:
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@@
 			)
 		)
-		(property "Footprint" ""
+		(property "Footprint" "JKC_Library:Display_HP_5082-7300"
 			(at 128.27 100.33 0)
 			(effects
@@
 				(path "/25ded3d7-7fc5-4a73-82e8-c02ba32fe53a/9c3e6a6e-1bd7-4020-9c43-ff5dae6e50b0"
 					(reference "U11")
+					(unit 1)
+				)
+			)
+			(project "displayDriver"
+				(path "/fa7d4c5f-4bdf-4b04-831b-f46410c303db"
+					(reference "U?")
 					(unit 1)
 				)
@@
 		(dnp no)
 		(fields_autoplaced yes)
-		(property "Reference" "#PWR035"
+		(property "Reference" "#PWR037"
 			(at 128.27 86.36 0)
 			(effects
@@
 			(project "AC_Clock"
 				(path "/25ded3d7-7fc5-4a73-82e8-c02ba32fe53a/8415622f-d6a3-4b8d-9ccc-26640cae3420"
-					(reference "#PWR035")
+					(reference "#PWR037")
 					(unit 1)
 				)
 				(path "/25ded3d7-7fc5-4a73-82e8-c02ba32fe53a/866e8215-1d8c-47c5-8153-911fecd2aea2"
+					(reference "#PWR043")
+					(unit 1)
+				)
+				(path "/25ded3d7-7fc5-4a73-82e8-c02ba32fe53a/8bbb75c9-62b8-4128-b141-2203322cccf0"
+					(reference "#PWR039")
+					(unit 1)
+				)
+				(path "/25ded3d7-7fc5-4a73-82e8-c02ba32fe53a/9c3e6a6e-1bd7-4020-9c43-ff5dae6e50b0"
 					(reference "#PWR041")
 					(unit 1)
 				)
-				(path "/25ded3d7-7fc5-4a73-82e8-c02ba32fe53a/8bbb75c9-62b8-4128-b141-2203322cccf0"
-					(reference "#PWR037")
-					(unit 1)
-				)
-				(path "/25ded3d7-7fc5-4a73-82e8-c02ba32fe53a/9c3e6a6e-1bd7-4020-9c43-ff5dae6e50b0"
-					(reference "#PWR039")
+			)
+			(project "displayDriver"
+				(path "/fa7d4c5f-4bdf-4b04-831b-f46410c303db"
+					(reference "#PWR?")
 					(unit 1)
 				)
@@
 		(dnp no)
 		(fields_autoplaced yes)
-		(property "Reference" "#PWR036"
+		(property "Reference" "#PWR038"
 			(at 128.27 125.73 0)
 			(effects
@@
 			(project "AC_Clock"
 				(path "/25ded3d7-7fc5-4a73-82e8-c02ba32fe53a/8415622f-d6a3-4b8d-9ccc-26640cae3420"
-					(reference "#PWR036")
+					(reference "#PWR038")
 					(unit 1)
 				)
 				(path "/25ded3d7-7fc5-4a73-82e8-c02ba32fe53a/866e8215-1d8c-47c5-8153-911fecd2aea2"
+					(reference "#PWR044")
+					(unit 1)
+				)
+				(path "/25ded3d7-7fc5-4a73-82e8-c02ba32fe53a/8bbb75c9-62b8-4128-b141-2203322cccf0"
+					(reference "#PWR040")
+					(unit 1)
+				)
+				(path "/25ded3d7-7fc5-4a73-82e8-c02ba32fe53a/9c3e6a6e-1bd7-4020-9c43-ff5dae6e50b0"
 					(reference "#PWR042")
 					(unit 1)
 				)
-				(path "/25ded3d7-7fc5-4a73-82e8-c02ba32fe53a/8bbb75c9-62b8-4128-b141-2203322cccf0"
-					(reference "#PWR038")
-					(unit 1)
-				)
-				(path "/25ded3d7-7fc5-4a73-82e8-c02ba32fe53a/9c3e6a6e-1bd7-4020-9c43-ff5dae6e50b0"
-					(reference "#PWR040")
-					(unit 1)
-				)
-			)
-		)
-	)
+			)
+			(project "displayDriver"
+				(path "/fa7d4c5f-4bdf-4b04-831b-f46410c303db"
+					(reference "#PWR?")
+					(unit 1)
+				)
+			)
+		)
+	)
+	(sheet_instances
+		(path "/"
+			(page "1")
+		)
+	)
+	(embedded_fonts no)
 )
